File: MultiBoardMini_HW.kicad_pcb (KiCad board)
At the start: 2 copper layers, 63 x 63 mm, 56 parts, among them J1 PB0, J2 PA10, J3 Conn_01x02_Male, J4 PA10, J6 Conn_01x04, SW1 PF1, SW2 RESET, SW3 SW_Push_DPDT, SW5 SW_Push_DPDT, T3 PTS_1.5_2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

Commit message: オートルート前のほぼ完成
Parts:
- removed REF3 (x4): MountingHole_3.2mm_M3, MountingHole:MountingHole_3.2mm_M3
Routing:
- added copper zone on B.Cu, net GND
- added copper zone on F.Cu, net GND
Changed lines of the file:
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@@
     )
   )
-  (footprint "MountingHole:MountingHole_3.2mm_M3" (layer "F.Cu")
-    (at 27.5 -27.5)
-    (descr "Mounting Hole 3.2mm, no annular, M3")
-    (tags "mounting hole 3.2mm no annular m3")
-    (attr exclude_from_pos_files exclude_from_bom)
-    (fp_text reference "REF3" (at 0 -4.2) (layer "F.SilkS") hide
-        (effects (font (size 1 1) (thickness 0.15)))
-    )
-    (fp_text value "MountingHole_3.2mm_M3" (at 0 4.2) (layer "F.Fab") hide
-        (effects (font (size 1 1) (thickness 0.15)))
-    )
-    (fp_text user "${REFERENCE}" (at 0.3 0) (layer "F.Fab") hide
-        (effects (font (size 1 1) (thickness 0.15)))
-    )
-    (fp_circle (center 0 0) (end 3.2 0)
-      (stroke (width 0.15) (type solid)) (fill none) (layer "Cmts.User"))
-    (fp_circle (center 0 0) (end 3.45 0)
-      (stroke (width 0.05) (type solid)) (fill none) (layer "F.CrtYd"))
-    (pad "" np_thru_hole circle (at 0 0) (size 3.2 3.2) (drill 3.2) (layers "F&B.Cu" "*.Mask"))
-  )
-  (footprint "MountingHole:MountingHole_3.2mm_M3" (layer "F.Cu")
-    (at -27.5 -27.5)
-    (descr "Mounting Hole 3.2mm, no annular, M3")
-    (tags "mounting hole 3.2mm no annular m3")
-    (attr exclude_from_pos_files exclude_from_bom)
-    (fp_text reference "REF3" (at 0 -4.2) (layer "F.SilkS") hide
-        (effects (font (size 1 1) (thickness 0.15)))
-    )
-    (fp_text value "MountingHole_3.2mm_M3" (at 0 4.2) (layer "F.Fab") hide
-        (effects (font (size 1 1) (thickness 0.15)))
-    )
-    (fp_text user "${REFERENCE}" (at 0.3 0) (layer "F.Fab") hide
-        (effects (font (size 1 1) (thickness 0.15)))
-    )
-    (fp_circle (center 0 0) (end 3.2 0)
-      (stroke (width 0.15) (type solid)) (fill none) (layer "Cmts.User"))
-    (fp_circle (center 0 0) (end 3.45 0)
-      (stroke (width 0.05) (type solid)) (fill none) (layer "F.CrtYd"))
-    (pad "" np_thru_hole circle (at 0 0) (size 3.2 3.2) (drill 3.2) (layers "F&B.Cu" "*.Mask"))
-  )
   (footprint "Connector_JST:JST_XA_B04B-XASK-1_1x04_P2.50mm_Vertical" (layer "F.Cu")
     (at -10.5 -6.855 180)
@@
     )
   )
-  (footprint "MountingHole:MountingHole_3.2mm_M3" (layer "F.Cu")
-    (at -27.5 27.5)
-    (descr "Mounting Hole 3.2mm, no annular, M3")
-    (tags "mounting hole 3.2mm no annular m3")
-    (attr exclude_from_pos_files exclude_from_bom)
-    (fp_text reference "REF3" (at 0 -4.2) (layer "F.SilkS") hide
-        (effects (font (size 1 1) (thickness 0.15)))
-    )
-    (fp_text value "MountingHole_3.2mm_M3" (at 0 4.2) (layer "F.Fab") hide
-        (effects (font (size 1 1) (thickness 0.15)))
-    )
-    (fp_text user "${REFERENCE}" (at 0.3 0) (layer "F.Fab") hide
-        (effects (font (size 1 1) (thickness 0.15)))
-    )
-    (fp_circle (center 0 0) (end 3.2 0)
-      (stroke (width 0.15) (type solid)) (fill none) (layer "Cmts.User"))
-    (fp_circle (center 0 0) (end 3.45 0)
-      (stroke (width 0.05) (type solid)) (fill none) (layer "F.CrtYd"))
-    (pad "" np_thru_hole circle (at 0 0) (size 3.2 3.2) (drill 3.2) (layers "F&B.Cu" "*.Mask"))
-  )
   (footprint "MultiBoardMini_Libraries:PTS_1.5_2" (layer "F.Cu")
     (at 0 26)
@@
     )
   )
-  (footprint "MountingHole:MountingHole_3.2mm_M3" (layer "F.Cu")
-    (at 27.5 27.5)
-    (descr "Mounting Hole 3.2mm, no annular, M3")
-    (tags "mounting hole 3.2mm no annular m3")
-    (attr exclude_from_pos_files exclude_from_bom)
-    (fp_text reference "REF3" (at 0 -4.2) (layer "F.SilkS") hide
-        (effects (font (size 1 1) (thickness 0.15)))
-    )
-    (fp_text value "MountingHole_3.2mm_M3" (at 0 4.2) (layer "F.Fab") hide
-        (effects (font (size 1 1) (thickness 0.15)))
-    )
-    (fp_text user "${REFERENCE}" (at 0.3 0) (layer "F.Fab") hide
-        (effects (font (size 1 1) (thickness 0.15)))
-    )
-    (fp_circle (center 0 0) (end 3.2 0)
-      (stroke (width 0.15) (type solid)) (fill none) (layer "Cmts.User"))
-    (fp_circle (center 0 0) (end 3.45 0)
-      (stroke (width 0.05) (type solid)) (fill none) (layer "F.CrtYd"))
-    (pad "" np_thru_hole circle (at 0 0) (size 3.2 3.2) (drill 3.2) (layers "F&B.Cu" "*.Mask"))
-  )
   (footprint "MultiBoardMini_Libraries:PTS_1.5_2" (layer "F.Cu")
     (at -11 26)
@@
   (segment (start -8.5 26) (end -10.35 27.85) (width 1.3) (layer "F.Cu") (net 51))
   (segment (start -9.25 -20.355) (end -9.25 -16.855) (width 0.5) (layer "B.Cu") (net 62))
+  (zone (net 2) (net_name "GND") (layers "F&B.Cu") (hatch edge 0.5)
+    (connect_pads (clearance 0.5))
+    (min_thickness 0.25) (filled_areas_thickness no)
+    (fill (thermal_gap 0.5) (thermal_bridge_width 0.5))
+    (polygon
+      (pts
+        (xy 23.5 -24.5)
+        (xy 31 -16.5)
+        (xy 31 16.5)
+        (xy 16.5 31)
+        (xy -16 31)
+        (xy -31 16)
+        (xy -31 -13.5)
+        (xy -20 -24.5)
+      )
+    )
+  )
 )

Commit message: Autoroute 前の完成だと思われるもの
Routing:
- net +3V3: track 64.5 -> 84.7 mm
Changed lines of the file:
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@@
   (segment (start 7 2.04) (end 7 2.518324) (width 1.75) (layer "B.Cu") (net 2))
   (segment (start -5.25 -18.355) (end -7.25 -20.355) (width 0.5) (layer "B.Cu") (net 3))
+  (segment (start 3.736396 -24) (end 2 -24) (width 0.5) (layer "B.Cu") (net 3))
   (segment (start -7.25 -10.355) (end -7.25 -11.105) (width 0.5) (layer "B.Cu") (net 3))
   (segment (start -7.25 -0.355) (end -5.25 -2.355) (width 0.5) (layer "B.Cu") (net 3))
+  (segment (start 2 -24) (end 2 -21.65) (width 0.5) (layer "B.Cu") (net 3))
   (segment (start -5.605 -22) (end -0.936396 -22) (width 0.5) (layer "B.Cu") (net 3))
   (segment (start 19.2 -15.35) (end 19.2 -23.036396) (width 0.5) (layer "B.Cu") (net 3))
@@
   (segment (start -18.12 12.385) (end -13.392206 12.385) (width 0.5) (layer "B.Cu") (net 3))
   (segment (start -7.25 -11.105) (end -5.25 -13.105) (width 0.5) (layer "B.Cu") (net 3))
+  (segment (start 18 -23.9) (end 3.836396 -23.9) (width 0.5) (layer "B.Cu") (net 3))
   (segment (start -5.25 1.645) (end -7.25 -0.355) (width 0.5) (layer "B.Cu") (net 3))
   (segment (start 18.75 -14.9) (end 19.2 -15.35) (width 0.5) (layer "B.Cu") (net 3))
+  (segment (start 3.836396 -23.9) (end 3.736396 -24) (width 0.5) (layer "B.Cu") (net 3))
   (segment (start 18 -14.9) (end 18.75 -14.9) (width 0.5) (layer "B.Cu") (net 3))
   (segment (start -5.25 4.242794) (end -5.25 1.645) (width 0.5) (layer "B.Cu") (net 3))
   (segment (start 18.336396 -23.9) (end 18 -23.9) (width 0.5) (layer "B.Cu") (net 3))
   (segment (start -13.392206 12.385) (end -5.25 4.242794) (width 0.5) (layer "B.Cu") (net 3))
+  (segment (start 1.25 -20.9) (end 0.5 -20.9) (width 0.5) (layer "B.Cu") (net 3))
   (segment (start 0.163604 -20.9) (end 0.5 -20.9) (width 0.5) (layer "B.Cu") (net 3))
   (segment (start -5.25 -2.355) (end -5.25 -8.355) (width 0.5) (layer "B.Cu") (net 3))
   (segment (start 19.2 -23.036396) (end 18.336396 -23.9) (width 0.5) (layer "B.Cu") (net 3))
+  (segment (start 2 -21.65) (end 1.25 -20.9) (width 0.5) (layer "B.Cu") (net 3))
   (segment (start -5.25 -13.105) (end -5.25 -18.355) (width 0.5) (layer "B.Cu") (net 3))
   (segment (start -0.936396 -22) (end 0.163604 -20.9) (width 0.5) (layer "B.Cu") (net 3))
