File: MultiBoardMini_HW.kicad_sch (KiCad schematic)
At the start: 52 parts, among them J1 PB0, J2 PA10, J3 Conn_01x02_Male, J6 Conn_01x04, SW1 PF1, SW2 RESET, SW3 SW_Push_DPDT, SW5 SW_Push_DPDT, T1 PTS_1.5_2, T3 PTS_1.5_2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

Commit message: 部品は一おおむね完了
Parts:
- SW1, SW2: footprint Button_Switch_THT:SW_PUSH_6mm_H4.3mm -> Button_Switch_SMD:SW_Push_1P1T_NO_6x6mm_H9.5mm
Connections:
- net GND: now also U3.9 (GND); no longer J1.1 (Pin_1), J2.1 (Pin_1)
- new net GNDPWR: J1.1 (Pin_1), J2.1 (Pin_1)
- no-connect marks 23 -> 22

Commit message: PWR　MOT 配線一旦できた
Connections:
- net GNDPWR is gone; now on net GND: J1.1 (Pin_1), J2.1 (Pin_1)

Commit message: 改良版の電源配線暫定版
Parts:
- added JP1: Jumper_NC_Dual, Jumper:SolderJumper-3_P2.0mm_Open_TrianglePad1.0x1.5mm, symbol Device:Jumper_NC_Dual
- PA1, PA2, PWR1: footprint LED_SMD:LED_1206_3216Metric_Pad1.42x1.75mm_HandSolder -> LED_SMD:LED_0805_2012Metric_Pad1.15x1.40mm_HandSolder
- SW1, SW2: footprint Button_Switch_SMD:SW_Push_1P1T_NO_6x6mm_H9.5mm -> Button_Switch_THT:SW_PUSH_6mm
- SW3, SW5: footprint MultiBoardMini_Libraries:SSSS213202 -> MultiBoardMini_Libraries:IS-2235
- SW4: footprint Button_Switch_SMD:SW_Push_1P1T_NO_Vertical_Wuerth_434133025816 -> Button_Switch_THT:SW_PUSH_1P1T_6x3.5mm_H4.3_APEM_MJTP1243
Connections:
- net +5V: now also JP1.3
- net PWR: now also JP1.1; no longer J1.2 (Pin_2), J2.2 (Pin_2)
- new net: J1.2 (Pin_2), J2.2 (Pin_2), JP1.2
Changed lines of the file:
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@@
   (junction (at 167.64 124.46) (diameter 0) (color 0 0 0 0)
   )
-  (junction (at 419.1 288.29) (diameter 0) (color 0 0 0 0)
+  (junction (at 414.02 288.29) (diameter 0) (color 0 0 0 0)
   )
   (junction (at 375.92 127) (diameter 0) (color 0 0 0 0)
@@
     (stroke (width 0) (type default))
   )
+  (wire (pts (xy 416.56 280.67) (xy 416.56 281.94))
+    (stroke (width 0) (type default))
+  )
   (wire (pts (xy 247.65 295.91) (xy 247.65 311.15))
     (stroke (width 0) (type default))
@@
     (stroke (width 0) (type default))
   )
+  (wire (pts (xy 435.61 294.64) (xy 435.61 279.4))
+    (stroke (width 0) (type default))
+  )
   (wire (pts (xy 510.54 154.94) (xy 510.54 151.13))
     (stroke (width 0) (type default))
   )
+  (wire (pts (xy 416.56 280.67) (xy 424.18 280.67))
+    (stroke (width 0) (type default))
+  )
   (wire (pts (xy 402.59 116.84) (xy 402.59 121.92))
     (stroke (width 0) (type default))
@@
     (stroke (width 0) (type default))
   )
-  (wire (pts (xy 419.1 288.29) (xy 419.1 302.26))
+  (wire (pts (xy 427.355 227.33) (xy 433.07 227.33))
     (stroke (width 0) (type default))
   )
-  (wire (pts (xy 427.355 227.33) (xy 433.07 227.33))
+  (wire (pts (xy 424.18 280.67) (xy 424.18 279.4))
     (stroke (width 0) (type default))
   )
@@
     (stroke (width 0) (type default))
   )
-  (wire (pts (xy 340.36 185.42) (xy 177.8 185.42))
+  (wire (pts (xy 340.36 180.34) (xy 177.8 180.34))
     (stroke (width 0) (type default))
   )
@@
     (stroke (width 0) (type default))
   )
-  (wire (pts (xy 419.1 280.67) (xy 419.1 288.29))
-    (stroke (width 0) (type default))
-  )
   (wire (pts (xy 66.04 187.96) (xy 77.47 187.96))
     (stroke (width 0) (type default))
@@
     (stroke (width 0) (type default))
   )
-  (wire (pts (xy 419.1 302.26) (xy 411.48 302.26))
-    (stroke (width 0) (type default))
-  )
   (wire (pts (xy 330.2 132.08) (xy 320.04 132.08))
     (stroke (width 0) (type default))
@@
     (stroke (width 0) (type default))
   )
+  (wire (pts (xy 414.02 302.26) (xy 411.48 302.26))
+    (stroke (width 0) (type default))
+  )
   (wire (pts (xy 307.34 146.05) (xy 307.34 147.32))
     (stroke (width 0) (type default))
@@
     (stroke (width 0) (type default))
   )
-  (wire (pts (xy 340.36 240.03) (xy 340.36 185.42))
+  (wire (pts (xy 340.36 240.03) (xy 340.36 180.34))
     (stroke (width 0) (type default))
   )
@@
     (stroke (width 0) (type default))
   )
-  (wire (pts (xy 410.21 288.29) (xy 419.1 288.29))
+  (wire (pts (xy 410.21 288.29) (xy 414.02 288.29))
     (stroke (width 0) (type default))
   )
@@
     (stroke (width 0) (type default))
   )
+  (wire (pts (xy 416.56 294.64) (xy 435.61 294.64))
+    (stroke (width 0) (type default))
+  )
   (wire (pts (xy 238.76 290.83) (xy 309.88 290.83))
     (stroke (width 0) (type default))
@@
     (stroke (width 0) (type default))
   )
+  (wire (pts (xy 414.02 288.29) (xy 414.02 302.26))
+    (stroke (width 0) (type default))
+  )
   (wire (pts (xy 292.1 328.93) (xy 292.1 326.39))
     (stroke (width 0) (type default))
@@
     (stroke (width 0) (type default))
   )
-  (wire (pts (xy 177.8 185.42) (xy 177.8 129.54))
+  (wire (pts (xy 177.8 180.34) (xy 177.8 129.54))
     (stroke (width 0) (type default))
   )
@@
     )
   )
-  (global_label "PWR" (shape input) (at 419.1 280.67 90) (fields_autoplaced)
+  (global_label "PWR" (shape input) (at 424.18 279.4 90) (fields_autoplaced)
     (effects (font (size 1.27 1.27)) (justify left))
-    (property "Intersheetrefs" "${INTERSHEET_REFS}" (at -31.75 424.18 0)
+    (property "Intersheetrefs" "${INTERSHEET_REFS}" (at -26.67 422.91 0)
       (effects (font (size 1.27 1.27)) hide)
     )
@@
     )
   )
+  (netclass_flag "" (length 2.54) (shape round) (at 414.02 302.26 270) (fields_autoplaced)
+    (effects (font (size 1.27 1.27)) (justify right bottom))
+    (property "Netclass" "MOTOR" (at 416.56 301.5615 90)
+      (effects (font (size 1.27 1.27) italic) (justify left))
+    )
+  )
+  (netclass_flag "" (length 2.54) (shape round) (at 416.56 280.67 0) (fields_autoplaced)
+    (effects (font (size 1.27 1.27)) (justify left bottom))
+    (property "Netclass" "MOTOR" (at 417.2585 278.13 0)
+      (effects (font (size 1.27 1.27) italic) (justify left))
+    )
+  )
   (symbol (lib_id "Device:Jumper") (at 307.34 116.84 90) (unit 1)
     (in_bom yes) (on_board yes) (dnp no)
@@
       (effects (font (size 1.27 1.27)) (justify right) hide)
     )
-    (property "Footprint" "LED_SMD:LED_1206_3216Metric_Pad1.42x1.75mm_HandSolder" (at 303.9872 335.2292 90)
+    (property "Footprint" "LED_SMD:LED_0805_2012Metric_Pad1.15x1.40mm_HandSolder" (at 303.9872 335.2292 90)
       (effects (font (size 1.27 1.27)) (justify right) hide)
     )
@@
       (effects (font (size 1.27 1.27)))
     )
-    (property "Footprint" "Button_Switch_SMD:SW_Push_1P1T_NO_6x6mm_H9.5mm" (at 250.19 261.62 0)
+    (property "Footprint" "Button_Switch_THT:SW_PUSH_6mm" (at 250.19 261.62 0)
       (effects (font (size 1.27 1.27)) hide)
     )
@@
     )
   )
+  (symbol (lib_id "power:+5V") (at 435.61 279.4 0) (unit 1)
+    (in_bom yes) (on_board yes) (dnp no)
+    (property "Reference" "#PWR011" (at 435.61 283.21 0)
+      (effects (font (size 1.27 1.27)) hide)
+    )
+    (property "Value" "+5V" (at 435.991 275.0058 0)
+      (effects (font (size 1.27 1.27)))
+    )
+    (property "Footprint" "" (at 435.61 279.4 0)
+      (effects (font (size 1.27 1.27)) hide)
+    )
+    (property "Datasheet" "" (at 435.61 279.4 0)
+      (effects (font (size 1.27 1.27)) hide)
+    )
+    (pin "1")
+    (instances
+      (project "MultiBoardMini"
+        (path "/7b4d6a3e-dec4-4756-807e-679f9b6d01df"
+          (reference "#PWR011") (unit 1)
+        )
+      )
+      (project "MultiBoardMini_HW"
+        (path "/f89d8039-fb4d-432a-bf6a-fadbc30a6f09"
+          (reference "#PWR06") (unit 1)
+        )
+      )
+    )
+  )
   (symbol (lib_id "power:GND") (at 167.64 153.67 0) (unit 1)
     (in_bom yes) (on_board yes) (dnp no)
@@
       (effects (font (size 1.27 1.27)) (justify right))
     )
-    (property "Footprint" "Button_Switch_SMD:SW_Push_1P1T_NO_6x6mm_H9.5mm" (at 242.57 261.62 0)
+    (property "Footprint" "Button_Switch_THT:SW_PUSH_6mm" (at 242.57 261.62 0)
       (effects (font (size 1.27 1.27)) hide)
     )
@@
       (effects (font (size 1.27 1.27)) (justify right))
     )
-    (property "Footprint" "LED_SMD:LED_1206_3216Metric_Pad1.42x1.75mm_HandSolder" (at 312.8772 335.2292 90)
+    (property "Footprint" "LED_SMD:LED_0805_2012Metric_Pad1.15x1.40mm_HandSolder" (at 312.8772 335.2292 90)
       (effects (font (size 1.27 1.27)) (justify right) hide)
     )
@@
       (effects (font (size 1.27 1.27)))
     )
-    (property "Footprint" "MultiBoardMini_Libraries:SSSS213202" (at 504.19 215.9 0)
+    (property "Footprint" "MultiBoardMini_Libraries:IS-2235" (at 504.19 215.9 0)
       (effects (font (size 1.27 1.27)) hide)
     )
@@
       (effects (font (size 1.27 1.27)) (justify right))
     )
-    (property "Footprint" "Button_Switch_SMD:SW_Push_1P1T_NO_Vertical_Wuerth_434133025816" (at 412.115 204.47 0)
+    (property "Footprint" "Button_Switch_THT:SW_PUSH_1P1T_6x3.5mm_H4.3_APEM_MJTP1243" (at 412.115 204.47 0)
       (effects (font (size 1.27 1.27)) hide)
     )
@@
       (effects (font (size 1.27 1.27)))
     )
-    (property "Footprint" "MultiBoardMini_Libraries:SSSS213202" (at 354.33 275.59 0)
+    (property "Footprint" "MultiBoardMini_Libraries:IS-2235" (at 354.33 275.59 0)
       (effects (font (size 1.27 1.27)) hide)
     )
@@
       (effects (font (size 1.27 1.27)) (justify right))
     )
-    (property "Footprint" "LED_SMD:LED_1206_3216Metric_Pad1.42x1.75mm_HandSolder" (at 295.0972 335.2292 90)
+    (property "Footprint" "LED_SMD:LED_0805_2012Metric_Pad1.15x1.40mm_HandSolder" (at 295.0972 335.2292 90)
       (effects (font (size 1.27 1.27)) (justify right) hide)
     )
@@
         )
       )
+    )
+  )
+  (symbol (lib_id "Device:Jumper_NC_Dual") (at 416.56 288.29 270) (unit 1)
+    (in_bom yes) (on_board yes) (dnp no)
+    (property "Reference" "JP1" (at 419.1508 289.4584 90)
+      (effects (font (size 1.27 1.27)) (justify left))
+    )
+    (property "Value" "Jumper_NC_Dual" (at 419.1508 287.147 90)
+      (effects (font (size 1.27 1.27)) (justify left))
+    )
+    (property "Footprint" "Jumper:SolderJumper-3_P2.0mm_Open_TrianglePad1.0x1.5mm" (at 419.1508 285.9786 90)
+      (effects (font (size 1.27 1.27)) (justify left) hide)
+    )
+    (property "Datasheet" "~" (at 416.56 288.29 0)
+      (effects (font (size 1.27 1.27)) hide)
+    )
+    (pin "1")
+    (pin "2")
+    (pin "3")
+    (instances
+      (project "MultiBoardMini"
+        (path "/7b4d6a3e-dec4-4756-807e-679f9b6d01df"
+          (reference "JP1") (unit 1)
+        )
+      )
+      (project "MultiBoardMini_HW"
+        (path "/f89d8039-fb4d-432a-bf6a-fadbc30a6f09"
+          (reference "JP4") (unit 1)
+        )
+      )

Commit message: esp32変更
Parts:
- removed U3: ESP32-C3-WROOM-02-N4, MultiBoardMini_Libraries:ESP-WROOM-02, symbol ESP32-C3-WROOM-02-N4:ESP32-C3-WROOM-02-N4
- added U7: ESP32-WROOM-32, RF_Module:ESP32-WROOM-32, symbol RF_Module:ESP32-WROOM-32
Connections:
- net +3V3: now also U7.2 (VDD)
- net GND: now also U7.1 (GND), U7.15 (GND), U7.38 (GND), U7.39 (GND)
- net at J6.2 (Pin_2): now also U7.34 (RXD0/IO3); no longer U2.3_1 (PA9)
- net at J6.1 (Pin_1): now also U7.35 (TXD0/IO1); no longer U2.3_2 (PA10)
- net at C2.1, D1.2 (A), R9.1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: now also U7.3 (EN)
- net at R10.1, SW3.2 (B), SW3.5 (B): now also U7.25 (IO0)
- new net rx: U2.3_1 (PA9)
- new net tx: U2.3_2 (PA10)
- no-connect marks 22 -> 18
Other:
- moved on the sheet: J6

Commit message: 回路図 ESP32の回路修正完了
Connections:
- net rx is gone; now on an unnamed net: U2.3_1 (PA9)
- net tx is gone; now on an unnamed net: U2.3_2 (PA10)
Changed lines of the file:
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@@
+    (stroke (width 0) (type default))
+  )
+  (wire (pts (xy 381 255.27) (xy 448.31 255.27))
     (stroke (width 0) (type default))
   )
@@
     (stroke (width 0) (type default))
   )
-  (wire (pts (xy 381 255.27) (xy 402.59 255.27))
-    (stroke (width 0) (type default))
-  )
   (wire (pts (xy 128.27 187.96) (xy 134.62 187.96))
     (stroke (width 0) (type default))
@@
     (stroke (width 0) (type default))
   )
+  (wire (pts (xy 383.54 252.73) (xy 449.58 252.73))
+    (stroke (width 0) (type default))
+  )
   (wire (pts (xy 215.9 287.02) (xy 215.9 271.78))
     (stroke (width 0) (type default))
@@
     (stroke (width 0) (type default))
   )
+  (wire (pts (xy 485.14 283.21) (xy 449.58 283.21))
+    (stroke (width 0) (type default))
+  )
+  (wire (pts (xy 485.14 237.49) (xy 485.14 283.21))
+    (stroke (width 0) (type default))
+  )
+  (wire (pts (xy 482.6 237.49) (xy 485.14 237.49))
+    (stroke (width 0) (type default))
+  )
   (wire (pts (xy 238.76 280.67) (xy 247.65 280.67))
     (stroke (width 0) (type default))
@@
     (stroke (width 0) (type default))
   )
-  (wire (pts (xy 402.59 247.65) (xy 402.59 252.73))
-    (stroke (width 0) (type default))
-  )
   (wire (pts (xy 359.41 278.13) (xy 363.22 278.13))
     (stroke (width 0) (type default))
@@
     (stroke (width 0) (type default))
   )
+  (wire (pts (xy 448.31 284.48) (xy 448.31 255.27))
+    (stroke (width 0) (type default))
+  )
   (wire (pts (xy 190.5 127) (xy 175.26 127))
     (stroke (width 0) (type default))
@@
     (stroke (width 0) (type default))
   )
+  (wire (pts (xy 482.6 234.95) (xy 486.41 234.95))
+    (stroke (width 0) (type default))
+  )
   (wire (pts (xy 455.93 127) (xy 482.6 127))
     (stroke (width 0) (type default))
@@
     (stroke (width 0) (type default))
   )
+  (wire (pts (xy 486.41 234.95) (xy 486.41 284.48))
+    (stroke (width 0) (type default))
+  )
   (wire (pts (xy 275.59 242.57) (xy 275.59 303.53))
     (stroke (width 0) (type default))
@@
     (stroke (width 0) (type default))
   )
-  (wire (pts (xy 402.59 255.27) (xy 402.59 259.08))
-    (stroke (width 0) (type default))
-  )
   (wire (pts (xy 500.38 154.94) (xy 510.54 154.94))
     (stroke (width 0) (type default))
@@
     (stroke (width 0) (type default))
   )
+  (wire (pts (xy 486.41 284.48) (xy 448.31 284.48))
+    (stroke (width 0) (type default))
+  )
   (wire (pts (xy 328.93 227.33) (xy 335.28 227.33))
     (stroke (width 0) (type default))
@@
     (stroke (width 0) (type default))
   )
-  (wire (pts (xy 383.54 252.73) (xy 402.59 252.73))
-    (stroke (width 0) (type default))
-  )
   (wire (pts (xy 450.85 124.46) (xy 450.85 154.94))
     (stroke (width 0) (type default))
@@
   )
   (wire (pts (xy 190.5 132.08) (xy 180.34 132.08))
+    (stroke (width 0) (type default))
+  )
+  (wire (pts (xy 449.58 283.21) (xy 449.58 252.73))
     (stroke (width 0) (type default))
   )
@@
     )
   )
-  (global_label "tx" (shape input) (at 402.59 247.65 0) (fields_autoplaced)
-    (effects (font (size 1.27 1.27)) (justify left))
-    (property "Intersheetrefs" "${INTERSHEET_REFS}" (at 407.329 247.65 0)
-      (effects (font (size 1.27 1.27)) (justify left) hide)
-    )
-  )
   (global_label "GND" (shape input) (at 226.06 157.48 0) (fields_autoplaced)
     (effects (font (size 1.27 1.27)) (justify left))
@@
       (effects (font (size 1.27 1.27)) (justify left) hide)
     )
-  )
-  (global_label "rx" (shape input) (at 402.59 259.08 0) (fields_autoplaced)
-    (effects (font (size 1.27 1.27)) (justify left))
-    (property "Intersheetrefs" "${INTERSHEET_REFS}" (at 407.3895 259.08 0)
-      (effects (font (size 1.27 1.27)) (justify left) hide)
-    )
