File: MultiBoardMini_HW.kicad_sch (KiCad schematic)
At the start: 54 parts, among them J1 PB0, J2 PA10, J3 Conn_01x02_Male, J6 Conn_01x04, SW1 PF1, SW2 RESET, SW3 SW_Push_DPDT, SW5 SW_Push_DPDT, T1 PTS_1.5_2, T3 PTS_1.5_2, U2 NUCLEO-F303K8, U3 M78AR5-1, U4 TB67H303HG, U5 TB67H303HG, U6 MCP2562-E_SN, U7 ESP32-WROOM-32

Commit message: V0.41試作発注用完成 PCB ASSEMBLY用BOM、positionデータ追加
Parts:
- removed D1: D, Diode_SMD:D_SOD-123F, symbol Device:D
- C4: KCSC (none) -> C1711
- C4: LCSC (none) -> C1711
- U7: LCSC (none) -> C529581
Connections:
- net GND is gone; now on net +5V: C1.2, C10.2, C2.2, C4.2, C4.2, C4.2, C4.2, C5.2, C5.2, C9.2, CAN1.1 (Pin_1), ENC/IO_1.1 (Pin_1), ENC/IO_2.1 (Pin_1), IO_1.1 (Pin_1), J1.1 (Pin_1), J2.1 (Pin_1), J3.2 (Pin_2), J6.3 (Pin_3), R2.1, R2.1, R3.2, R3.2, R4.1, R5.1, R6.1, SW1.1, SW2.1, SW3.3 (C), SW3.6 (C), SW4.1, SW5.3 (C), SW5.6 (C), T3.P$1, U2.3_4 (GND_1), U2.4_2 (GND_2), U3.2 (GND), U4.11 (RSB), U4.13 (PGNDB), U4.15 (RSA), U4.17 (PGNDA), U4.18 (TEST2), U4.19 (TEST3), U4.2 (SGND), U4.21 (TEST4), U4.3 (SELECT), U4.4 (TEST1), U4.5 (VREF), U5.11 (RSB), U5.13 (PGNDB), U5.15 (RSA), U5.17 (PGNDA), U5.18 (TEST2), U5.19 (TEST3), U5.2 (SGND), U5.21 (TEST4), U5.3 (SELECT), U5.4 (TEST1), U5.5 (VREF), U6.2 (VSS), U6.8 (STBY), U7.1 (GND), U7.15 (GND), U7.38 (GND), U7.39 (GND)
Changed lines of the file:
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@@
     (stroke (width 0) (type default))
   )
-  (wire (pts (xy 426.72 294.64) (xy 426.72 295.91))
-    (stroke (width 0) (type default))
-  )
   (wire (pts (xy 510.54 154.94) (xy 510.54 151.13))
     (stroke (width 0) (type default))
@@
     (stroke (width 0) (type default))
   )
-  (wire (pts (xy 426.72 303.53) (xy 426.72 304.8))
+  (wire (pts (xy 426.72 294.64) (xy 426.72 304.8))
     (stroke (width 0) (type default))
   )
@@
       (project "MultiBoardMini_HW"
         (path "/f89d8039-fb4d-432a-bf6a-fadbc30a6f09"
-          (reference "PA7") (unit 1)
+          (reference "L2") (unit 1)
         )
       )
@@
       (effects (font (size 1.27 1.27)) hide)
     )
+    (property "LCSC" "C529581" (at 467.36 240.03 0)
+      (effects (font (size 1.27 1.27)) hide)
+    )
     (pin "1")
     (pin "10")
@@
       (project "MultiBoardMini_HW"
         (path "/f89d8039-fb4d-432a-bf6a-fadbc30a6f09"
-          (reference "PA6") (unit 1)
+          (reference "L3") (unit 1)
         )
       )
@@
       (effects (font (size 1.27 1.27)) hide)
     )
+    (property "KCSC" "C1711" (at 254 118.11 0)
+      (effects (font (size 1.27 1.27)) hide)
+    )
     (pin "1")
     (pin "2")
@@
     )
   )
-  (symbol (lib_id "Device:D") (at 426.72 299.72 270) (unit 1)
-    (in_bom yes) (on_board yes) (dnp no) (fields_autoplaced)
-    (property "Reference" "D1" (at 429.26 298.45 90)
-      (effects (font (size 1.27 1.27)) (justify left))
-    )
-    (property "Value" "D" (at 429.26 300.99 90)
-      (effects (font (size 1.27 1.27)) (justify left))
-    )
-    (property "Footprint" "Diode_SMD:D_SOD-123F" (at 426.72 299.72 0)
-      (effects (font (size 1.27 1.27)) hide)
-    )
-    (property "Datasheet" "~" (at 426.72 299.72 0)
-      (effects (font (size 1.27 1.27)) hide)
-    )
-    (property "Sim.Device" "D" (at 426.72 299.72 0)
-      (effects (font (size 1.27 1.27)) hide)
-    )
-    (property "Sim.Pins" "1=K 2=A" (at 426.72 299.72 0)
-      (effects (font (size 1.27 1.27)) hide)
-    )
-    (pin "1")
-    (pin "2")
-    (instances
-      (project "MultiBoardMini"
-        (path "/7b4d6a3e-dec4-4756-807e-679f9b6d01df"
-          (reference "D1") (unit 1)
-        )
-      )
-      (project "MultiBoardMini_HW"
-        (path "/f89d8039-fb4d-432a-bf6a-fadbc30a6f09"
-          (reference "D2") (unit 1)
-        )
-      )
-    )
-  )
   (symbol (lib_id "Switch:SW_Push_DPDT") (at 504.19 220.98 0) (unit 1)
     (in_bom yes) (on_board yes) (dnp no) (fields_autoplaced)
@@
       (effects (font (size 1.27 1.27)) hide)
     )
+    (property "LCSC" "C1711" (at 262.89 113.03 0)
+      (effects (font (size 1.27 1.27)) hide)
+    )
     (pin "1")
     (pin "2")
@@
       (project "MultiBoardMini_HW"
         (path "/f89d8039-fb4d-432a-bf6a-fadbc30a6f09"
-          (reference "PWR1") (unit 1)
+          (reference "L1") (unit 1)
         )
       )

Commit message: とりあえず保存
Parts:
- C9: value 4.7μF -> 3.3μF
- SW1, SW2: footprint Button_Switch_SMD:SW_Push_1P1T_NO_6x6mm_H9.5mm -> MultiBoardMini_Libraries:SW_TL3301FF160QG
Changed lines of the file:
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@@
       (effects (font (size 1.27 1.27)))
     )
-    (property "Footprint" "Button_Switch_SMD:SW_Push_1P1T_NO_6x6mm_H9.5mm" (at 250.19 261.62 0)
+    (property "Footprint" "MultiBoardMini_Libraries:SW_TL3301FF160QG" (at 250.19 261.62 0)
       (effects (font (size 1.27 1.27)) hide)
     )
@@
       (effects (font (size 1.27 1.27)) (justify right))
     )
-    (property "Footprint" "Button_Switch_SMD:SW_Push_1P1T_NO_6x6mm_H9.5mm" (at 242.57 261.62 0)
+    (property "Footprint" "MultiBoardMini_Libraries:SW_TL3301FF160QG" (at 242.57 261.62 0)
       (effects (font (size 1.27 1.27)) hide)
     )
@@
       (effects (font (size 1.27 1.27)) (justify left))
     )
-    (property "Value" "4.7μF" (at 513.461 148.463 0)
+    (property "Value" "3.3μF" (at 513.461 148.463 0)
       (effects (font (size 1.27 1.27)) (justify left))
     )

Commit message: GNDと5V+がつながっていた問題を解消
Connections:
- net +5V: no longer C1.2, C10.2, C2.2, C4.2, C4.2, C4.2, C4.2, C5.2, C5.2, C9.2, CAN1.1 (Pin_1), ENC/IO_1.1 (Pin_1), ENC/IO_2.1 (Pin_1), IO_1.1 (Pin_1), J1.1 (Pin_1), J2.1 (Pin_1), J3.2 (Pin_2), J6.3 (Pin_3), R2.1, R2.1, R3.2, R3.2, R4.1, R5.1, R6.1, SW1.1, SW2.1, SW3.3 (C), SW3.6 (C), SW4.1, SW5.3 (C), SW5.6 (C), T3.P$1, U2.3_4 (GND_1), U2.4_2 (GND_2), U3.2 (GND), U4.11 (RSB), U4.13 (PGNDB), U4.15 (RSA), U4.17 (PGNDA), U4.18 (TEST2), U4.19 (TEST3), U4.2 (SGND), U4.21 (TEST4), U4.3 (SELECT), U4.4 (TEST1), U4.5 (VREF), U5.11 (RSB), U5.13 (PGNDB), U5.15 (RSA), U5.17 (PGNDA), U5.18 (TEST2), U5.19 (TEST3), U5.2 (SGND), U5.21 (TEST4), U5.3 (SELECT), U5.4 (TEST1), U5.5 (VREF), U6.2 (VSS), U6.8 (STBY), U7.1 (GND), U7.15 (GND), U7.38 (GND), U7.39 (GND)
- new net GND: C1.2, C10.2, C2.2, C4.2, C4.2, C4.2, C4.2, C5.2, C5.2, C9.2, CAN1.1 (Pin_1), ENC/IO_1.1 (Pin_1), ENC/IO_2.1 (Pin_1), IO_1.1 (Pin_1), J1.1 (Pin_1), J2.1 (Pin_1), J3.2 (Pin_2), J6.3 (Pin_3), R2.1, R2.1, R3.2, R3.2, R4.1, R5.1, R6.1, SW1.1, SW2.1, SW3.3 (C), SW3.6 (C), SW4.1, SW5.3 (C), SW5.6 (C), T3.P$1, U2.3_4 (GND_1), U2.4_2 (GND_2), U3.2 (GND), U4.11 (RSB), U4.13 (PGNDB), U4.15 (RSA), U4.17 (PGNDA), U4.18 (TEST2), U4.19 (TEST3), U4.2 (SGND), U4.21 (TEST4), U4.3 (SELECT), U4.4 (TEST1), U4.5 (VREF), U5.11 (RSB), U5.13 (PGNDB), U5.15 (RSA), U5.17 (PGNDA), U5.18 (TEST2), U5.19 (TEST3), U5.2 (SGND), U5.21 (TEST4), U5.3 (SELECT), U5.4 (TEST1), U5.5 (VREF), U6.2 (VSS), U6.8 (STBY), U7.1 (GND), U7.15 (GND), U7.38 (GND), U7.39 (GND)
Changed lines of the file:
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@@
   (junction (at 224.79 287.02) (diameter 0) (color 0 0 0 0)
   )
-  (junction (at 411.48 304.8) (diameter 0) (color 0 0 0 0)
-  )
   (junction (at 499.11 215.9) (diameter 0) (color 0 0 0 0)
   )
@@
   )
   (junction (at 276.86 109.22) (diameter 0) (color 0 0 0 0)
-  )
-  (junction (at 426.72 294.64) (diameter 0) (color 0 0 0 0)
   )
   (junction (at 402.59 121.92) (diameter 0) (color 0 0 0 0)
@@
     (stroke (width 0) (type default))
   )
-  (wire (pts (xy 411.48 304.8) (xy 426.72 304.8))
-    (stroke (width 0) (type default))
-  )
   (wire (pts (xy 236.22 127) (xy 236.22 119.38))
     (stroke (width 0) (type default))
@@
     (stroke (width 0) (type default))
   )
-  (wire (pts (xy 426.72 294.64) (xy 439.42 294.64))
-    (stroke (width 0) (type default))
-  )
   (wire (pts (xy 238.76 295.91) (xy 247.65 295.91))
     (stroke (width 0) (type default))
@@
     (stroke (width 0) (type default))
   )
-  (wire (pts (xy 416.56 294.64) (xy 426.72 294.64))
+  (wire (pts (xy 416.56 294.64) (xy 439.42 294.64))
     (stroke (width 0) (type default))
   )
@@
     (stroke (width 0) (type default))
   )
-  (wire (pts (xy 426.72 294.64) (xy 426.72 304.8))
-    (stroke (width 0) (type default))
-  )
