File: UGOKU-One.kicad_sch (KiCad schematic)
At the start: 52 parts, among them J2 Conn_02x03_Odd_Even, J2 PA10, J3 Conn_01x02_Male, J6 Conn_01x04, SW1 PF1, SW2 RESET, SW3 SW_Push_DPDT, SW5 SW_Push_DPDT, T1 PTS_1.5_2, T3 PTS_1.5_2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

Commit message: saisinban(XA仕様)
Parts:
- R4: value 3.3k -> 510
- R5, R6: value 3.3k -> 1k
Changed lines of the file:
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@@
       (effects (font (size 1.27 1.27)) (justify right))
     )
-    (property "Value" "3.3k" (at 302.768 341.503 0)
+    (property "Value" "1k" (at 302.768 341.503 0)
       (effects (font (size 1.27 1.27)) (justify right))
     )
@@
       (effects (font (size 1.27 1.27)) (justify right))
     )
-    (property "Value" "3.3k" (at 293.878 341.503 0)
+    (property "Value" "510" (at 293.878 341.503 0)
       (effects (font (size 1.27 1.27)) (justify right))
     )
@@
       (effects (font (size 1.27 1.27)) (justify right))
     )
-    (property "Value" "3.3k" (at 311.658 341.503 0)
-      (effects (font (size 1.27 1.27)) (justify right))
-    )
+    (property "Value" "1k" (at 311.658 341.503 0)
+      (effects (font (size 1.27 1.27)) (justify right))
+    )
